Commit message: Imported upstream version '1.0.5' of 'upstream'

File: configs/urdf/qbhand.urdf (robot description, URDF)
Before this commit: robot qbhand, 38 links, 37 joints
Links:
- link qbhand_index_middle_link: geometry collision mesh filename=package://qb_hand_description/meshes/ph_short_collision.stl scale=0.001 0.001 0.001; visual mesh filename=package://qb_hand_description/meshes/ph_short.stl scale=0.001 0.001 0.001
- link qbhand_little_middle_link: geometry collision mesh filename=package://qb_hand_description/meshes/ph_short_collision.stl scale=0.001 0.001 0.001; visual mesh filename=package://qb_hand_description/meshes/ph_short.stl scale=0.001 0.001 0.001
- link qbhand_little_proximal_link: geometry collision mesh filename=package://qb_hand_description/meshes/ph_short_collision.stl scale=0.001 0.001 0.001; visual mesh filename=package://qb_hand_description/meshes/ph_short.stl scale=0.001 0.001 0.001
- link qbhand_middle_middle_link: geometry collision mesh filename=package://qb_hand_description/meshes/ph_short_collision.stl scale=0.001 0.001 0.001; visual mesh filename=package://qb_hand_description/meshes/ph_short.stl scale=0.001 0.001 0.001
- link qbhand_ring_middle_link: geometry collision mesh filename=package://qb_hand_description/meshes/ph_short_collision.stl scale=0.001 0.001 0.001; visual mesh filename=package://qb_hand_description/meshes/ph_short.stl scale=0.001 0.001 0.001
- link qbhand_thumb_proximal_link: geometry collision mesh filename=package://qb_hand_description/meshes/ph_short_collision.stl scale=0.001 0.001 0.001; visual mesh filename=package://qb_hand_description/meshes/ph_short.stl scale=0.001 0.001 0.001
